Commit message: Upgrade camera to RGB-D

File: catkin_ws/src/my_robot/urdf/my_robot.xacro (robot description, xacro)
@@ -131,5 +131,5 @@
   </joint>
   <!-- Camera -->
-  <link name="camera">
+  <link name="camera_link">
     <collision name='camera_collision'>
       <origin xyz="0 0 0" rpy="0 0 0"/>
@@ -154,5 +154,5 @@
     </visual>
   </link>
-  <gazebo reference="camera">
+  <gazebo reference="camera_link">
     <material>Gazebo/Yellow</material>
   </gazebo>
@@ -160,8 +160,15 @@
   <joint type="fixed" name="camera_joint">
     <origin xyz="0.3 0 0" rpy="0 0 0"/>
-    <child link="camera"/>
-    <parent link="chassis"/>
-    <axis xyz="0 1 0" rpy="0 0 0"/>
-  </joint>
+    <child link="camera_link"/>
+    <parent link="chassis"/>
+    <axis xyz="0 1 0" rpy="0 0 0"/>
+  </joint>
+  <joint name="camera_optical_joint" type="fixed">
+    <origin xyz="0 0 0" rpy="-1.5707 0 -1.5707"/>
+    <parent link="camera_link"/>
+    <child link="camera_link_optical"/>
+  </joint>
+  <link name="camera_link_optical">
+  </link>
   <!-- Lidar -->
   <link name="hokuyo">
